Commit message: Update mercury_x1.urdf

File: src/turn_on_mercury_robot/urdf/mercury_x1/mercury_x1.urdf (robot description, URDF)
Before this commit: robot firefighter, 19 links, 18 joints
Links:
- link base_link: geometry collision mesh filename=package://turn_on_mercury_robot/urdf/mercury_x1/base.dae; visual mesh filename=package://turn_on_mercury_robot/urdf/mercury_x1/base.dae
- link link1_L: geometry collision mesh filename=package://turn_on_mercury_robot/urdf/mercury_x1/joint1_L.dae; visual mesh filename=package://turn_on_mercury_robot/urdf/mercury_x1/joint1_L.dae
- link link1_R: geometry collision mesh filename=package://turn_on_mercury_robot/urdf/mercury_x1/joint1_R.dae; visual mesh filename=package://turn_on_mercury_robot/urdf/mercury_x1/joint1_R.dae
- link link2_L: geometry collision mesh filename=package://turn_on_mercury_robot/urdf/mercury_x1/joint2_L.dae; visual mesh filename=package://turn_on_mercury_robot/urdf/mercury_x1/joint2_L.dae
- link link2_R: geometry collision mesh filename=package://turn_on_mercury_robot/urdf/mercury_x1/joint2_R.dae; visual mesh filename=package://turn_on_mercury_robot/urdf/mercury_x1/joint2_R.dae
- link link3_L: geometry collision mesh filename=package://turn_on_mercury_robot/urdf/mercury_x1/joint3_L.dae; visual mesh filename=package://turn_on_mercury_robot/urdf/mercury_x1/joint3_L.dae
- link link3_R: geometry collision mesh filename=package://turn_on_mercury_robot/urdf/mercury_x1/joint3_R.dae; visual mesh filename=package://turn_on_mercury_robot/urdf/mercury_x1/joint3_R.dae
- link link4_L: geometry collision mesh filename=package://turn_on_mercury_robot/urdf/mercury_x1/joint4_L.dae; visual mesh filename=package://turn_on_mercury_robot/urdf/mercury_x1/joint4_L.dae
- link link4_R: geometry collision mesh filename=package://turn_on_mercury_robot/urdf/mercury_x1/joint4_R.dae; visual mesh filename=package://turn_on_mercury_robot/urdf/mercury_x1/joint4_R.dae
- link link5_L: geometry collision mesh filename=package://turn_on_mercury_robot/urdf/mercury_x1/joint5_L.dae; visual mesh filename=package://turn_on_mercury_robot/urdf/mercury_x1/joint5_L.dae
- link link5_R: geometry collision mesh filename=package://turn_on_mercury_robot/urdf/mercury_x1/joint5_R.dae; visual mesh filename=package://turn_on_mercury_robot/urdf/mercury_x1/joint5_R.dae
- link link6_L: geometry collision mesh filename=package://turn_on_mercury_robot/urdf/mercury_x1/joint6_L.dae; visual mesh filename=package://turn_on_mercury_robot/urdf/mercury_x1/joint6_L.dae
- link link6_R: geometry collision mesh filename=package://turn_on_mercury_robot/urdf/mercury_x1/joint6_R.dae; visual mesh filename=package://turn_on_mercury_robot/urdf/mercury_x1/joint6_R.dae
- link link7_L: geometry collision mesh filename=package://turn_on_mercury_robot/urdf/mercury_x1/joint7_L.dae; visual mesh filename=package://turn_on_mercury_robot/urdf/mercury_x1/joint7_L.dae
- link link7_R: geometry collision mesh filename=package://turn_on_mercury_robot/urdf/mercury_x1/joint7_R.dae; visual mesh filename=package://turn_on_mercury_robot/urdf/mercury_x1/joint7_R.dae
- link link_body: geometry collision mesh filename=package://turn_on_mercury_robot/urdf/mercury_x1/body.dae; visual mesh filename=package://turn_on_mercury_robot/urdf/mercury_x1/body.dae
- link link_eye: geometry collision mesh filename=package://turn_on_mercury_robot/urdf/mercury_x1/head_eye.dae; visual mesh filename=package://turn_on_mercury_robot/urdf/mercury_x1/head_eye.dae
- link link_head: geometry collision mesh filename=package://turn_on_mercury_robot/urdf/mercury_x1/head.dae; visual mesh filename=package://turn_on_mercury_robot/urdf/mercury_x1/head.dae
