Commit message: Update mercury_x1.urdf joint limit

File: turn_on_mercury_robot/urdf/mercury_x1/mercury_x1.urdf (robot description, URDF)
Before this commit: robot firefighter, 19 links, 18 joints
Joints:
- joint eye: limit lower=0 upper=0.83 effort=1000.0 velocity=0 -> lower=-1.04 upper=0 effort=1000.0 velocity=0
- joint head: limit lower=-2.4085 upper=3.2812 effort=1000.0 velocity=0 -> lower=-2.321 upper=3.2812 effort=1000.0 velocity=0
- joint joint1_L: limit lower=-3.1066 upper=3.1066 effort=1000.0 velocity=0 -> lower=-2.879 upper=2.879 effort=1000.0 velocity=0
- joint joint1_R: limit lower=-3.1066 upper=3.1066 effort=1000.0 velocity=0 -> lower=-2.879 upper=2.879 effort=1000.0 velocity=0
- joint joint2_L: limit lower=-1.4311 upper=2.2689 effort=1000.0 velocity=0 -> lower=-0.959 upper=1.658 effort=1000.0 velocity=0
- joint joint2_R: limit lower=-1.4311 upper=2.2689 effort=1000.0 velocity=0 -> lower=-0.959 upper=1.658 effort=1000.0 velocity=0
- joint joint3_L: limit lower=-3.1066 upper=3.1066 effort=1000.0 velocity=0 -> lower=-2.879 upper=2.879 effort=1000.0 velocity=0
- joint joint3_R: limit lower=-3.1066 upper=3.1066 effort=1000.0 velocity=0 -> lower=-2.879 upper=2.879 effort=1000.0 velocity=0
- joint joint4_L: limit lower=-3.0543 upper=0.2617 effort=1000.0 velocity=0 -> lower=-3.019 upper=0.087 effort=1000.0 velocity=0
- joint joint4_R: limit lower=-3.0543 upper=0.2617 effort=1000.0 velocity=0 -> lower=-3.019 upper=0.087 effort=1000.0 velocity=0
- joint joint5_L: limit lower=-3.1066 upper=3.1066 effort=1000.0 velocity=0 -> lower=-2.879 upper=2.879 effort=1000.0 velocity=0
- joint joint5_R: limit lower=-3.1066 upper=3.1066 effort=1000.0 velocity=0 -> lower=-2.879 upper=2.879 effort=1000.0 velocity=0
- joint joint7_L: limit lower=-3.1066 upper=3.1066 effort=1000.0 velocity=0 -> lower=-3.14 upper=3.14 effort=1000.0 velocity=0
- joint joint7_R: limit lower=-3.1066 upper=3.1066 effort=1000.0 velocity=0 -> lower=-3.14 upper=3.14 effort=1000.0 velocity=0

Commit message: 更新水星X1 URDF关节限位

File: turn_on_mercury_robot/urdf/mercury_x1/mercury_x1.urdf (robot description, URDF)
Before this commit: robot firefighter, 19 links, 18 joints
Joints:
- joint joint1_L: limit lower=-3.1066 upper=3.1066 effort=1000.0 velocity=0 -> lower=-2.879 upper=2.879 effort=1000.0 velocity=0
- joint joint1_R: limit lower=-3.1066 upper=3.1066 effort=1000.0 velocity=0 -> lower=-2.879 upper=2.879 effort=1000.0 velocity=0
- joint joint2_L: limit lower=-1.4311 upper=2.2689 effort=1000.0 velocity=0 -> lower=-0.8726 upper=2.0943 effort=1000.0 velocity=0
- joint joint2_R: limit lower=-1.4311 upper=2.2689 effort=1000.0 velocity=0 -> lower=-0.8726 upper=2.0943 effort=1000.0 velocity=0
- joint joint3_L: limit lower=-3.1066 upper=3.1066 effort=1000.0 velocity=0 -> lower=-2.879 upper=2.879 effort=1000.0 velocity=0
- joint joint3_R: limit lower=-3.1066 upper=3.1066 effort=1000.0 velocity=0 -> lower=-2.879 upper=2.879 effort=1000.0 velocity=0
- joint joint4_L: limit lower=-3.0543 upper=0.2617 effort=1000.0 velocity=0 -> lower=-2.879 upper=0.087 effort=1000.0 velocity=0
- joint joint4_R: limit lower=-3.0543 upper=0.2617 effort=1000.0 velocity=0 -> lower=-2.879 upper=0.087 effort=1000.0 velocity=0
- joint joint5_L: limit lower=-3.1066 upper=3.1066 effort=1000.0 velocity=0 -> lower=-2.879 upper=2.879 effort=1000.0 velocity=0
- joint joint5_R: limit lower=-3.1066 upper=3.1066 effort=1000.0 velocity=0 -> lower=-2.879 upper=2.879 effort=1000.0 velocity=0
- joint joint6_L: limit lower=-0.0349 upper=2.9321 effort=1000.0 velocity=0 -> lower=-0.3490 upper=4.6251 effort=1000.0 velocity=0
- joint joint6_R: limit lower=-0.0349 upper=2.9321 effort=1000.0 velocity=0 -> lower=-0.3490 upper=4.6251 effort=1000.0 velocity=0
- joint joint7_L: limit lower=-3.1066 upper=3.1066 effort=1000.0 velocity=0 -> lower=-3.14 upper=3.14 effort=1000.0 velocity=0
- joint joint7_R: limit lower=-3.1066 upper=3.1066 effort=1000.0 velocity=0 -> lower=-3.14 upper=3.14 effort=1000.0 velocity=0

Commit message: 更新X1 urdf J6初始姿态，优化滑块控制

File: turn_on_mercury_robot/urdf/mercury_x1/mercury_x1.urdf (robot description, URDF)
Before this commit: robot firefighter, 19 links, 18 joints
Joints:
- joint joint6_L: limit lower=-0.3490 upper=4.6251 effort=1000.0 velocity=0 -> lower=-1.9198 upper=3.0543 effort=1000.0 velocity=0; origin xyz= 0 0 0.08 rpy=1.5708 0 0 -> xyz= 0 0 0.08 rpy=1.5708 -1.5708 0
- joint joint6_R: limit lower=-0.3490 upper=4.6251 effort=1000.0 velocity=0 -> lower=-1.9198 upper=3.0543 effort=1000.0 velocity=0; origin xyz= 0 0 0.08 rpy=1.5708 0 0 -> xyz= 0 0 0.08 rpy=1.5708 -1.5708 0

Commit message: update ros1 code

File: turn_on_mercury_robot/urdf/mercury_x1/mercury_x1.urdf (robot description, URDF)
Before this commit: robot firefighter, 19 links, 18 joints
Joints:
- joint eye: limit lower=-1.04 upper=0 effort=1000.0 velocity=0 -> lower=0 upper=0.83 effort=1000.0 velocity=0
- joint head: limit lower=-2.321 upper=3.2812 effort=1000.0 velocity=0 -> lower=-2.4085 upper=3.2812 effort=1000.0 velocity=0
- joint joint2_L: limit lower=-0.959 upper=1.658 effort=1000.0 velocity=0 -> lower=-0.8726 upper=2.0943 effort=1000.0 velocity=0
- joint joint2_R: limit lower=-0.959 upper=1.658 effort=1000.0 velocity=0 -> lower=-0.8726 upper=2.0943 effort=1000.0 velocity=0
- joint joint4_L: limit lower=-3.019 upper=0.087 effort=1000.0 velocity=0 -> lower=-2.879 upper=0.087 effort=1000.0 velocity=0
- joint joint4_R: limit lower=-3.019 upper=0.087 effort=1000.0 velocity=0 -> lower=-2.879 upper=0.087 effort=1000.0 velocity=0
- joint joint6_L: limit lower=-0.0349 upper=2.9321 effort=1000.0 velocity=0 -> lower=-1.9198 upper=3.0543 effort=1000.0 velocity=0; origin xyz= 0 0 0.08 rpy=1.5708 0 0 -> xyz= 0 0 0.08 rpy=1.5708 -1.5708 0
- joint joint6_R: limit lower=-0.0349 upper=2.9321 effort=1000.0 velocity=0 -> lower=-1.9198 upper=3.0543 effort=1000.0 velocity=0; origin xyz= 0 0 0.08 rpy=1.5708 0 0 -> xyz= 0 0 0.08 rpy=1.5708 -1.5708 0

Commit message: x1 urdf add quality info

File: turn_on_mercury_robot/urdf/mercury_x1/mercury_x1.urdf (robot description, URDF)
Before this commit: robot firefighter, 19 links, 18 joints
Links:
- link base_link: mass None -> 47.2640; geometry collision mesh filename=package://mercury_description/urdf/mercury_x1/base.dae; visual mesh filename=package://mercury_description/urdf/mercury_x1/base.dae
- link link1_L: mass None -> 0.784; geometry collision mesh filename=package://mercury_description/urdf/mercury_x1/joint1_L.dae; visual mesh filename=package://mercury_description/urdf/mercury_x1/joint1_L.dae
- link link1_R: mass None -> 0.784; geometry collision mesh filename=package://mercury_description/urdf/mercury_x1/joint1_R.dae; visual mesh filename=package://mercury_description/urdf/mercury_x1/joint1_R.dae
- link link2_L: mass None -> 0; geometry collision mesh filename=package://mercury_description/urdf/mercury_x1/joint2_L.dae; visual mesh filename=package://mercury_description/urdf/mercury_x1/joint2_L.dae
- link link2_R: mass None -> 0; geometry collision mesh filename=package://mercury_description/urdf/mercury_x1/joint2_R.dae; visual mesh filename=package://mercury_description/urdf/mercury_x1/joint2_R.dae
- link link3_L: mass None -> 0.824; geometry collision mesh filename=package://mercury_description/urdf/mercury_x1/joint3_L.dae; visual mesh filename=package://mercury_description/urdf/mercury_x1/joint3_L.dae
- link link3_R: mass None -> 0.824; geometry collision mesh filename=package://mercury_description/urdf/mercury_x1/joint3_R.dae; visual mesh filename=package://mercury_description/urdf/mercury_x1/joint3_R.dae
- link link4_L: mass None -> 0.7; geometry collision mesh filename=package://mercury_description/urdf/mercury_x1/joint4_L.dae; visual mesh filename=package://mercury_description/urdf/mercury_x1/joint4_L.dae
- link link4_R: mass None -> 0.7; geometry collision mesh filename=package://mercury_description/urdf/mercury_x1/joint4_R.dae; visual mesh filename=package://mercury_description/urdf/mercury_x1/joint4_R.dae
- link link5_L: mass None -> 0.508; geometry collision mesh filename=package://mercury_description/urdf/mercury_x1/joint5_L.dae; visual mesh filename=package://mercury_description/urdf/mercury_x1/joint5_L.dae
- link link5_R: mass None -> 0.508; geometry collision mesh filename=package://mercury_description/urdf/mercury_x1/joint5_R.dae; visual mesh filename=package://mercury_description/urdf/mercury_x1/joint5_R.dae
- link link6_L: mass None -> 0.398; geometry collision mesh filename=package://mercury_description/urdf/mercury_x1/joint6_L.dae; visual mesh filename=package://mercury_description/urdf/mercury_x1/joint6_L.dae
- link link6_R: mass None -> 0.398; geometry collision mesh filename=package://mercury_description/urdf/mercury_x1/joint6_R.dae; visual mesh filename=package://mercury_description/urdf/mercury_x1/joint6_R.dae
- link link7_L: mass None -> 0.393; geometry collision mesh filename=package://mercury_description/urdf/mercury_x1/joint7_L.dae; visual mesh filename=package://mercury_description/urdf/mercury_x1/joint7_L.dae
- link link7_R: mass None -> 0.393; geometry collision mesh filename=package://mercury_description/urdf/mercury_x1/joint7_R.dae; visual mesh filename=package://mercury_description/urdf/mercury_x1/joint7_R.dae
- link link_body: mass None -> 5.516; geometry collision mesh filename=package://mercury_description/urdf/mercury_x1/body.dae; visual mesh filename=package://mercury_description/urdf/mercury_x1/body.dae
- link link_eye: mass None -> 0; geometry collision mesh filename=package://mercury_description/urdf/mercury_x1/head_eye.dae; visual mesh filename=package://mercury_description/urdf/mercury_x1/head_eye.dae
- link link_head: mass None -> 0; geometry collision mesh filename=package://mercury_description/urdf/mercury_x1/head.dae; visual mesh filename=package://mercury_description/urdf/mercury_x1/head.dae

Commit message: x1 urdf add quality info

File: turn_on_mercury_robot/urdf/mercury_x1/mercury_x1.urdf (robot description, URDF)
Before this commit: robot firefighter, 19 links, 18 joints
Links:
- link base_link: mass None -> 47.2640
- link link1_L: mass None -> 0.784
- link link1_R: mass None -> 0.784
- link link2_L: mass None -> 0
- link link2_R: mass None -> 0
- link link3_L: mass None -> 0.824
- link link3_R: mass None -> 0.824
- link link4_L: mass None -> 0.7
- link link4_R: mass None -> 0.7
- link link5_L: mass None -> 0.508
- link link5_R: mass None -> 0.508
- link link6_L: mass None -> 0.398
- link link6_R: mass None -> 0.398
- link link7_L: mass None -> 0.393
- link link7_R: mass None -> 0.393
- link link_body: mass None -> 5.516
- link link_eye: mass None -> 0
- link link_head: mass None -> 0

Commit message: feat(X1-URDF): Add two left and right camera models to the head of the urdf model and update the coordinate axis

File: turn_on_mercury_robot/urdf/mercury_x1/mercury_x1.urdf (robot description, URDF)
Before this commit: robot firefighter, 19 links, 18 joints
Links:
- added link link_left_camera, mass 0; collision mesh filename=package://turn_on_mercury_robot/urdf/mercury_x1/left_camera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; visual mesh filename=package://turn_on_mercury_robot/urdf/mercury_x1/left_camera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
- added link link_right_camera, mass 0; collision mesh filename=package://turn_on_mercury_robot/urdf/mercury_x1/right_camer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; visual mesh filename=package://turn_on_mercury_robot/urdf/mercury_x1/right_camer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
- link link_eye: geometry collision mesh filename=package://turn_on_mercury_robot/urdf/mercury_x1/dual_hole_c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; visual mesh filename=package://turn_on_mercury_robot/urdf/mercury_x1/dual_hole_c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
Joints:
- added joint left_camera: type fixed, parent link_eye, child link_left_camera, origin xyz= 0.008 0 -0.027  rpy=0 0 0, axis  0 0 1, limit lower=-1.04 upper=0 effort=1000.0 velocity=0
- added joint right_camera: type fixed, parent link_eye, child link_right_camera, origin xyz= 0.008 0 0.033  rpy=0 0 0, axis  0 0 1, limit lower=-1.04 upper=0 effort=1000.0 velocity=0
